Commit message: add stl and configs

File: src/fanuc_m16ib_description/urdf/fanuc_m16ib_macro.urdf.xacro (robot description, xacro)
@@ -8,5 +8,5 @@
 <!--set some parameters with default values used by the macros (kinematics description, simulation and control)-->
 <!--#######################################################################################################################################-->
-  <xacro:macro name="diy_robotarm" params="
+  <xacro:macro name="fanuc_m16ib" params="
     name
     tf_prefix
@@ -70,12 +70,12 @@
         <origin xyz="0 0 0" rpy="0 0 0"/>
         <geometry>
-          <mesh filename="package://fanuc_m16ib_description/meshes/visual/link_1.stl" scale="0.001 0.001 0.001"/>
-        </geometry>
-        <material name="${tf_prefix}yellow"/>
-      </visual>
-      <collision>
-        <origin xyz="0 0 0" rpy = "0 0 0"/>
-        <geometry>
-          <mesh filename="package://fanuc_m16ib_description/meshes/collision/link_1.stl" scale="0.001 0.001 0.001"/>
+          <mesh filename="package://fanuc_m16ib_description/meshes/visual/link1.stl" scale="0.001 0.001 0.001"/>
+        </geometry>
+        <material name="${tf_prefix}yellow"/>
+      </visual>
+      <collision>
+        <origin xyz="0 0 0" rpy = "0 0 0"/>
+        <geometry>
+          <mesh filename="package://fanuc_m16ib_description/meshes/collision/link1.stl" scale="0.001 0.001 0.001"/>
         </geometry>
         <material name="${tf_prefix}red"/>
@@ -95,12 +95,12 @@
         <origin xyz="0 0 0" rpy="0 0 0"/>
         <geometry>
-          <mesh filename="package://fanuc_m16ib_description/meshes/visual/link_2.stl" scale="0.001 0.001 0.001"/>
-        </geometry>
-        <material name="${tf_prefix}yellow"/>
-      </visual>
-      <collision>
-        <origin xyz="0 0 0" rpy = "0 0 0"/>
-        <geometry>
-          <mesh filename="package://fanuc_m16ib_description/meshes/collision/link_2.stl" scale="0.001 0.001 0.001"/>
+          <mesh filename="package://fanuc_m16ib_description/meshes/visual/link2.stl" scale="0.001 0.001 0.001"/>
+        </geometry>
+        <material name="${tf_prefix}yellow"/>
+      </visual>
+      <collision>
+        <origin xyz="0 0 0" rpy = "0 0 0"/>
+        <geometry>
+          <mesh filename="package://fanuc_m16ib_description/meshes/collision/link2.stl" scale="0.001 0.001 0.001"/>
         </geometry>
         <material name="${tf_prefix}red"/>
@@ -120,12 +120,12 @@
         <origin xyz="0 0 0" rpy="0 0 0"/>
         <geometry>
-          <mesh filename="package://fanuc_m16ib_description/meshes/visual/link_3.stl" scale="0.001 0.001 0.001"/>
-        </geometry>
-        <material name="${tf_prefix}yellow"/>
-      </visual>
-      <collision>
-        <origin xyz="0 0 0" rpy = "0 0 0"/>
-        <geometry>
-          <mesh filename="package://fanuc_m16ib_description/meshes/collision/link_3.stl" scale="0.001 0.001 0.001"/>
+          <mesh filename="package://fanuc_m16ib_description/meshes/visual/link3.stl" scale="0.001 0.001 0.001"/>
+        </geometry>
+        <material name="${tf_prefix}yellow"/>
+      </visual>
+      <collision>
+        <origin xyz="0 0 0" rpy = "0 0 0"/>
+        <geometry>
+          <mesh filename="package://fanuc_m16ib_description/meshes/collision/link3.stl" scale="0.001 0.001 0.001"/>
         </geometry>
         <material name="${tf_prefix}red"/>
@@ -145,12 +145,12 @@
         <origin xyz="0 0 0" rpy="0 0 0"/>
         <geometry>
-          <mesh filename="package://fanuc_m16ib_description/meshes/visual/link_4.stl" scale="0.001 0.001 0.001"/>
-        </geometry>
-        <material name="${tf_prefix}yellow"/>
-      </visual>
-      <collision>
-        <origin xyz="0 0 0" rpy = "0 0 0"/>
-        <geometry>
-          <mesh filename="package://fanuc_m16ib_description/meshes/collision/link_4.stl" scale="0.001 0.001 0.001"/>
+          <mesh filename="package://fanuc_m16ib_description/meshes/visual/link4.stl" scale="0.001 0.001 0.001"/>
+        </geometry>
+        <material name="${tf_prefix}yellow"/>
+      </visual>
+      <collision>
+        <origin xyz="0 0 0" rpy = "0 0 0"/>
+        <geometry>
+          <mesh filename="package://fanuc_m16ib_description/meshes/collision/link4.stl" scale="0.001 0.001 0.001"/>
         </geometry>
         <material name="${tf_prefix}red"/>
@@ -170,12 +170,12 @@
         <origin xyz="0 0 0" rpy="0 0 0"/>
         <geometry>
-          <mesh filename="package://fanuc_m16ib_description/meshes/visual/link_5.stl" scale="0.001 0.001 0.001"/>
-        </geometry>
-        <material name="${tf_prefix}yellow"/>
-      </visual>
-      <collision>
-        <origin xyz="0 0 0" rpy = "0 0 0"/>
-        <geometry>
-          <mesh filename="package://fanuc_m16ib_description/meshes/collision/link_5.stl" scale="0.001 0.001 0.001"/>
+          <mesh filename="package://fanuc_m16ib_description/meshes/visual/link5.stl" scale="0.001 0.001 0.001"/>
+        </geometry>
+        <material name="${tf_prefix}yellow"/>
+      </visual>
+      <collision>
+        <origin xyz="0 0 0" rpy = "0 0 0"/>
+        <geometry>
+          <mesh filename="package://fanuc_m16ib_description/meshes/collision/link5.stl" scale="0.001 0.001 0.001"/>
         </geometry>
         <material name="${tf_prefix}red"/>
@@ -195,5 +195,5 @@
         <origin xyz="0 0 0" rpy="0 0 0"/>
         <geometry>
-          <mesh filename="package://fanuc_m16ib_description/meshes/visual/link_6.stl" scale="0.001 0.001 0.001"/>
+          <mesh filename="package://fanuc_m16ib_description/meshes/visual/link6.stl" scale="0.001 0.001 0.001"/>
         </geometry>
         <material name="${tf_prefix}grey"/>
@@ -202,5 +202,5 @@
         <origin xyz="0 0 0" rpy = "0 0 0"/>
         <geometry>
-          <mesh filename="package://fanuc_m16ib_description/meshes/collision/link_6.stl" scale="0.001 0.001 0.001"/>
+          <mesh filename="package://fanuc_m16ib_description/meshes/collision/link6.stl" scale="0.001 0.001 0.001"/>
         </geometry>
         <material name="${tf_prefix}red"/>

File: src/fanuc_m16ib_description/urdf/fanuc_m16ib_model.urdf.xacro (robot description, xacro)
@@ -14,5 +14,5 @@
     <xacro:arg name="tf_prefix" default=""/>
     <xacro:arg name="use_fake_hardware" default="false" />
-    <xacro:arg name="generate_ros2_control_tag" default_"false"/>
+    <xacro:arg name="generate_ros2_control_tag" default="false"/>
     <!-- ros2_control related parameters -->
     <!-- TODO -->
@@ -25,12 +25,13 @@
    <!-- create link fixed to the "world" -->
     <link name="world" />
-    <xacro:diy_robotarm
+    <xacro:fanuc_m16ib
         name="$(arg name)"
         tf_prefix="$(arg tf_prefix)"
         parent="world"
         use_fake_hardware="$(arg use_fake_hardware)"
+        generate_ros2_control_tag="$(arg generate_ros2_control_tag)"
         initial_positions="${xacro.load_yaml(initial_positions_file)}"
         >
         <origin xyz="0 0 0" rpy="0 0 0" />          <!-- position robot in the world -->
-    </xacro:diy_robotarm>
+    </xacro:fanuc_m16ib>
 </robot>

Commit message: finished urdf without collision meshes

File: src/fanuc_m16ib_description/urdf/fanuc_m16ib_macro.urdf.xacro (robot description, xacro)
@@ -59,9 +59,9 @@
     <!-- Joint 1 -->
     <joint name="${tf_prefix}joint1" type="revolute">
-        <origin xyz="0 0 0" rpy="0 0 0"/>
+        <origin xyz="0 0 0.245" rpy="0 0 0"/>
         <parent link="${tf_prefix}base_link"/>
         <child link="${tf_prefix}link_1"/>
         <axis xyz="0.0 0.0 1.0"/>
-        <limit lower="0" upper="0" velocity="0" effort="0"/>
+        <limit lower="-2.697" upper="2.697" velocity="2.88" effort="1000"/>
     </joint>
     <!-- Link1 -->
@@ -84,9 +84,9 @@
     <!-- Joint 2 -->
     <joint name="${tf_prefix}joint2" type="revolute">
-        <origin xyz="0 0 0" rpy="0 0 0"/>
+        <origin xyz="-0.143 0.15 0.28" rpy="1.5707 0 -1.5707"/>
         <parent link="${tf_prefix}link_1"/>
         <child link="${tf_prefix}link_2"/>
         <axis xyz="0.0 0.0 1.0"/>
-        <limit lower="0" upper="0" velocity="0" effort="0"/>
+        <limit lower="-1.5707" upper="2.9725" velocity="2.88" effort="1000"/>
     </joint>
     <!-- Link2 -->
@@ -109,9 +109,9 @@
     <!-- Joint 3 -->
     <joint name="${tf_prefix}joint3" type="revolute">
-        <origin xyz="0 0 0" rpy="0 0 0"/>
+        <origin xyz="0 0.770 0.0189" rpy="0 3.1415 0"/>
         <parent link="${tf_prefix}link_2"/>
         <child link="${tf_prefix}link_3"/>
         <axis xyz="0.0 0.0 1.0"/>
-        <limit lower="0" upper="0" velocity="0" effort="0"/>
+        <limit lower="-2.967" upper="5.061" velocity="3.05" effort="1000"/>
     </joint>
     <!-- Link3 -->
@@ -133,10 +133,10 @@
     </link>
     <!-- Joint 4 -->
-    <joint name="${tf_prefix}wrist_1" type="revolute">
-        <origin xyz="0 0 0" rpy="0 0 0"/>
+    <joint name="${tf_prefix}joint4" type="revolute">
+        <origin xyz="0.184575 0.099755 0.163294" rpy="0 -1.5707 0"/>
         <parent link="${tf_prefix}link_3"/>
         <child link="${tf_prefix}link_4"/>
         <axis xyz="0.0 0.0 1.0"/>
-        <limit lower="0" upper="0" velocity="0" effort="0"/>
+        <limit lower="-3.491" upper="3.491" velocity="6.11" effort="1000"/>
     </joint>
     <!-- Link4 -->
@@ -159,9 +159,9 @@
     <!-- Joint 5 -->
     <joint name="${tf_prefix}joint5" type="revolute">
-        <origin xyz="0 0 0" rpy="0 0 0"/>
+        <origin xyz="-0.04679 0 -0.55593" rpy="0 1.5707 0"/>
         <parent link="${tf_prefix}link_4"/>
         <child link="${tf_prefix}link_5"/>
         <axis xyz="0.0 0.0 1.0"/>
-        <limit lower="0" upper="0" velocity="0" effort="0"/>
+        <limit lower="-2.443" upper="2.443" velocity="5.93" effort="1000"/>
     </joint>
     <!-- Link5 -->
@@ -184,9 +184,9 @@
     <!-- Joint 6 -->
     <joint name="${tf_prefix}joint6" type="revolute">
-        <origin xyz="0 0 0" rpy="0 0 0"/>
+        <origin xyz="0.080645 0 0.044376" rpy="0 1.5707 0"/>
         <parent link="${tf_prefix}link_5"/>
         <child link="${tf_prefix}link_6"/>
         <axis xyz="0.0 0.0 1.0"/>
-        <limit lower="0" upper="0" velocity="0" effort="0"/>
+        <limit lower="-7.854" upper="7.854" velocity="9.08" effort="1000"/>
     </joint>
     <!-- Link6 = Flange -->
@@ -207,4 +207,12 @@
       </collision>
     </link>
+        <!-- Joint to Tool0/ Flange -->
+        <joint name="${tf_prefix}to_tool0" type="fixed">
+          <origin xyz="0 0 0.0196" rpy="0 0 0"/>
+          <parent link="${tf_prefix}link_6"/>
+          <child link="${tf_prefix}tool0"/>
+      </joint>
+      <!-- tool0 -->
+      <link name="${tf_prefix}tool0"/>
   </xacro:macro>
 </robot>

Commit message: add coupling of axis 2 and 3

File: src/fanuc_m16ib_description/urdf/fanuc_m16ib_macro.urdf.xacro (robot description, xacro)
@@ -107,8 +107,19 @@
       </collision>
     </link>
+    <!-- Joint 2_mimic -->
+    <joint name="${tf_prefix}joint2_mimic" type="revolute">
+        <mimic joint="${tf_prefix}joint2" multiplier="1" offset="0"/>
+        <origin xyz="0 0.770 0.0189" rpy="0 3.1415 0"/>
+        <parent link="${tf_prefix}link_2"/>
+        <child link="${tf_prefix}link_2_mimic"/>
+        <axis xyz="0.0 0.0 1.0"/>
+        <limit lower="-1.5707" upper="2.9725" velocity="2.88" effort="1000"/>
+    </joint>
+    <!-- Link2_mimic -->
+    <link name="${tf_prefix}link_2_mimic"/>
     <!-- Joint 3 -->
     <joint name="${tf_prefix}joint3" type="revolute">
-        <origin xyz="0 0.770 0.0189" rpy="0 3.1415 0"/>
-        <parent link="${tf_prefix}link_2"/>
+        <origin xyz="0 0 0" rpy="0 0 0"/>
+        <parent link="${tf_prefix}link_2_mimic"/>
         <child link="${tf_prefix}link_3"/>
         <axis xyz="0.0 0.0 1.0"/>

Commit message: kinematics tuner

File: src/fanuc_m16ib_description/urdf/fanuc_m16ib_macro.urdf.xacro (robot description, xacro)
@@ -82,5 +82,5 @@
       </collision>
     </link>
-    <!-- Joint 2 -->
+    <!-- Joint 2 <limit lower="-1.5707" upper="2.9725" velocity="2.88" effort="1000"/> -->
     <joint name="${tf_prefix}joint2" type="revolute">
         <origin xyz="-0.143 0.15 0.28" rpy="1.5707 0 -1.5707"/>
@@ -88,5 +88,5 @@
         <child link="${tf_prefix}link_2"/>
         <axis xyz="0.0 0.0 1.0"/>
-        <limit lower="-1.5707" upper="2.9725" velocity="2.88" effort="1000"/>
+        <limit lower="-1.0" upper="1.0" velocity="2.88" effort="1000"/>
     </joint>
     <!-- Link2 -->
@@ -168,5 +168,5 @@
       </collision>
     </link>
-    <!-- Joint 5 -->
+    <!-- Joint 5 <limit lower="-2.443" upper="2.443" velocity="5.93" effort="1000"/>-->
     <joint name="${tf_prefix}joint5" type="revolute">
         <origin xyz="-0.04679 0 -0.55593" rpy="0 1.5707 0"/>
@@ -174,5 +174,5 @@
         <child link="${tf_prefix}link_5"/>
         <axis xyz="0.0 0.0 1.0"/>
-        <limit lower="-2.443" upper="2.443" velocity="5.93" effort="1000"/>
+        <limit lower="-1.5707" upper="1.5707" velocity="5.93" effort="1000"/>
     </joint>
     <!-- Link5 -->
@@ -193,5 +193,5 @@
       </collision>
     </link>
-    <!-- Joint 6 -->
+    <!-- Joint 6 <limit lower="-7.854" upper="7.854" velocity="9.08" effort="1000"/> -->
     <joint name="${tf_prefix}joint6" type="revolute">
         <origin xyz="0.080645 0 0.044376" rpy="0 1.5707 0"/>
@@ -199,5 +199,5 @@
         <child link="${tf_prefix}link_6"/>
         <axis xyz="0.0 0.0 1.0"/>
-        <limit lower="-7.854" upper="7.854" velocity="9.08" effort="1000"/>
+        <limit lower="-3.1415" upper="3.1415" velocity="9.08" effort="1000"/>
     </joint>
     <!-- Link6 = Flange -->

Commit message: add camera frame with false calibration

File: src/fanuc_m16ib_description/urdf/fanuc_m16ib_macro.urdf.xacro (robot description, xacro)
@@ -39,9 +39,10 @@
         <parent link="${parent}"/>
         <child link="${tf_prefix}base_link"/>
+        <xacro:insert_block name="origin"/>
     </joint>
     <!-- Link0 = Base -->
     <link name="${tf_prefix}base_link">
-      <origin xyz="0 0 0"/>
-      <visual>
+      <visual>
+        <origin rpy="0 0 -1.5707"/>
         <geometry>
           <mesh filename="package://fanuc_m16ib_description/meshes/visual/base.stl" scale="0.001 0.001 0.001"/>
@@ -50,5 +51,5 @@
       </visual>
       <collision>
-        <origin xyz="0 0 0"/>
+        <origin xyz="0 0 -1.5707"/>
         <geometry>
           <mesh filename="package://fanuc_m16ib_description/meshes/collision/base.stl" scale="0.001 0.001 0.001"/>
@@ -59,5 +60,5 @@
     <!-- Joint 1 -->
     <joint name="${tf_prefix}joint1" type="revolute">
-        <origin xyz="0 0 0.245" rpy="0 0 0"/>
+        <origin xyz="0 0 0.245" rpy="0 0 -1.5707"/>
         <parent link="${tf_prefix}base_link"/>
         <child link="${tf_prefix}link_1"/>
@@ -218,12 +219,12 @@
       </collision>
     </link>
-        <!-- Joint to Tool0/ Flange -->
-        <joint name="${tf_prefix}to_tool0" type="fixed">
-          <origin xyz="0 0 0.0196" rpy="0 0 0"/>
-          <parent link="${tf_prefix}link_6"/>
-          <child link="${tf_prefix}tool0"/>
-      </joint>
-      <!-- tool0 -->
-      <link name="${tf_prefix}tool0"/>
+    <!-- Joint to Tool0/ Flange -->
+    <joint name="${tf_prefix}to_tool0" type="fixed">
+      <origin xyz="0 0 0.0196" rpy="0 0 0"/>
+      <parent link="${tf_prefix}link_6"/>
+      <child link="${tf_prefix}tool0"/>
+    </joint>
+    <!-- tool0 -->
+    <link name="${tf_prefix}tool0"/>
   </xacro:macro>
 </robot>

File: src/fanuc_m16ib_description/urdf/fanuc_m16ib_model.urdf.xacro (robot description, xacro)
@@ -5,7 +5,8 @@
     <xacro:arg name="name" default="fanuc_m16ib"/>
 <!--#######################################################################################################################################-->
-   <!-- import main macro -->
+   <!-- import macros -->
 <!--#######################################################################################################################################-->
     <xacro:include filename="$(find fanuc_m16ib_description)/urdf/fanuc_m16ib_macro.urdf.xacro"/>
+    <xacro:include filename="$(find fanuc_m16ib_description)/urdf/zivid.urdf.xacro"/>
 <!--#######################################################################################################################################-->
     <!-- set ros2 parameters, which will passsed to the macros-->
@@ -20,4 +21,7 @@
     <xacro:arg name="initial_positions_file" default="$(find fanuc_m16ib_description)/config/initial_positions.yaml"/>
     <xacro:property name="initial_positions_file" default="$(arg initial_positions_file)"/>
+    <!-- hand eye calibration -->
+    <xacro:arg name="hand_eye_file" default="$(find fanuc_m16ib_description)/config/hand_eye_calibration.yaml"/>
+    <xacro:property name="hand_eye_file" default="$(arg hand_eye_file)"/>
 <!--#######################################################################################################################################-->
    <!-- call the main macro by passing parameters to build the arm -->
@@ -35,3 +39,9 @@
         <origin xyz="0 0 0" rpy="0 0 0" />          <!-- position robot in the world -->
     </xacro:fanuc_m16ib>
+    <!-- add camera link with calibrated pose -->
+    <xacro:zivid_camera
+        parent="$(arg tf_prefix)base_link"
+        hand_eye ="${xacro.load_yaml(hand_eye_file)}"
+        >
+    </xacro:zivid_camera>
 </robot>
