Commit message: add octomap

File: src/fanuc_m16ib_moveit_config/srdf/fanuc_m16ib_macro.srdf.xacro (robot description, xacro)
@@ -15,5 +15,5 @@
     <!-- default configurations -->
     <group_state name="home" group="${name}">
-        <joint name="$(arg tf_prefix)joint1" value="0"/>
+        <joint name="$(arg tf_prefix)joint1" value="1.5707"/>
         <joint name="$(arg tf_prefix)joint2" value="0"/>
         <joint name="$(arg tf_prefix)joint3" value="0"/>
